File: RocciBoard.kicad_sch (KiCad schematic)
At the start: 193 parts, among them J1 Battery, J10 M3, J11 I2C6, J12 Power, J13 M2, J14 I2C7, J2 I2C0, J3 I2C1, J4 I2C2, J5 I2C3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

Commit message: final version V1.0
Parts:
- Q1: LCSC C693103 -> C2997
Changed lines of the file:
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@@
       (effects (font (size 1.27 1.27)) (justify left) hide)
     )
-    (property "LCSC" "C693103" (at 269.24 71.12 0)
+    (property "LCSC" "C2997" (at 269.24 71.12 0)
       (effects (font (size 1.27 1.27)) hide)
     )
