File: RocciBoard.kicad_pcb (KiCad board)
At the start: 2 copper layers, 99 x 54 mm, 215 parts, among them J1 Battery, J10 M3, J11 I2C6, J12 Power, J13 M2, J14 I2C7, J2 I2C0, J3 I2C1, J4 I2C2, J5 I2C3, J6 M0, J7 I2C4, J8 M1, J9 I2C5, Q1 IRF 7424, Q2 2N7002, SW1 SW_DIP_x01, U1 LMR33630, U10 LM317_TO-252, U11 CJ431, U12 CJ431, U2 LM317_TO-252, U3 LM317_TO-252, U4 TPS3700, U5 TCA9548A, U6 DRV8871, U7 DRV8871, U8 DRV8871, U9 DRV8871

Commit message: Version 1.2 finished
Parts:
- removed C22, C23: 100n, Capacitor_SMD:C_0603_1608Metric
- removed D32: SB10100L, Package_TO_SOT_SMD:TO-277A
- removed D33: BT137S-600E, Package_TO_SOT_SMD:TO-252-2
- removed F2: 10A, Fuse:Fuseholder_Cylinder-5x20mm_Wuerth_696103101002-SMD_Horizontal_Open
- removed R20: 240, Resistor_SMD:R_0603_1608Metric
- removed R24: 390, Resistor_SMD:R_0603_1608Metric
- removed R69: 1k5, Resistor_SMD:R_0603_1608Metric
- removed R70: 1k3, Resistor_SMD:R_0603_1608Metric
- removed R71: 1k, Resistor_SMD:R_0603_1608Metric
- removed R72: 2k, Resistor_SMD:R_0603_1608Metric
- removed U12: CJ431, Package_TO_SOT_SMD:SOT-23
- removed U2, U3: LM317_TO-252, Package_TO_SOT_SMD:TO-252-2
- added C24: 10nF, Capacitor_SMD:C_0603_1608Metric, F.Cu at (154.5, 93.1)
- added C25: 10nF, Capacitor_SMD:C_0603_1608Metric, F.Cu at (157.6, 95.3)
- added C26: 100nF, Capacitor_SMD:C_0603_1608Metric, F.Cu at (150.6, 93.1)
- added C27: 10nF, Capacitor_SMD:C_0603_1608Metric, F.Cu at (157.8, 99.5)
- added C28: 47pF, Capacitor_SMD:C_0603_1608Metric, F.Cu at (153.4, 102.3)
- added C29: 100nF, Capacitor_SMD:C_0603_1608Metric, F.Cu at (157.6, 91.9)
- added C30: 100nF, Capacitor_SMD:C_0603_1608Metric, F.Cu at (150.0, 102.3)
- added D26: 1N5819WS, Diode_SMD:D_SOD-323, F.Cu at (147.7, 90.5)
- added JP22: Jumper_2_Open, Jumper:SolderJumper-2_P1.3mm_Open_Pad1.0x1.5mm, B.Cu at (146.1, 100.9)
- added Q3: TM30N03D, Package_TO_SOT_SMD:TO-252-2, F.Cu at (151.2, 85.1)
- added R74: 4.7k, Resistor_SMD:R_0603_1608Metric, F.Cu at (148.1, 98.8)
- added R75: 51, Resistor_SMD:R_0603_1608Metric, F.Cu at (152.6, 93.1)
- added R76: 0, Resistor_SMD:R_0603_1608Metric, F.Cu at (157.6, 93.6)
- added R77: 100, Resistor_SMD:R_0603_1608Metric, F.Cu at (157.8, 97.9)
- added R78: 68k, Resistor_SMD:R_0603_1608Metric, F.Cu at (158.5, 102.3)
- added R79: 24k, Resistor_SMD:R_0603_1608Metric, F.Cu at (156.8, 102.3)
- added R80: 2.7k, Resistor_SMD:R_0603_1608Metric, F.Cu at (151.7, 102.3)
- added R81: 510k, Resistor_SMD:R_0603_1608Metric, F.Cu at (164.8, 100.9)
- added R82: 12k, Resistor_SMD:R_0603_1608Metric, F.Cu at (163.2, 100.9)
- added R83: 68k, Resistor_SMD:R_0603_1608Metric, F.Cu at (161.5, 100.9)
- added U13: TPS3700, Package_TO_SOT_SMD:SOT-23-6, F.Cu at (163.0, 97.6)
- added U14: AMS1117, Package_TO_SOT_SMD:SOT-223-3_TabPin2, F.Cu at (176.4, 90.2)
- Q1: value IRF 7424 -> TM30N03D; footprint Package_SO:SOIC-8_3.9x4.9mm_P1.27mm -> Package_TO_SOT_SMD:TO-252-2
- R13: value 4700k 1% -> 100k
- R14: value 10k -> 1mΩ 1%; footprint Resistor_SMD:R_0603_1608Metric -> Resistor_SMD:R_1206_3216Metric
- R17: value 620 -> 680
- R19: value 10k 1% -> 100k
- R21: value 240 -> 200
- R25: value 1k3 -> 1k
- R26: value 180k 1% -> 3.9k
- R65: value 1k -> 100k
- R66: value 240 -> 7,5k
- R67: value 720 -> 39k
- R68: value 1k -> 470k
- R7: value 24.9k -> 33k
- R73: value 9100k 1% -> 3.3k
- U10: value LM317_TO-252 -> TPS3700; footprint Package_TO_SOT_SMD:TO-252-2 -> Package_TO_SOT_SMD:SOT-23-6; moved to F.Cu
- U11: value CJ431 -> AMS1117-3.3; footprint Package_TO_SOT_SMD:SOT-23 -> Package_TO_SOT_SMD:SOT-223-3_TabPin2
- U4: value TPS3700 -> LM74900; footprint Package_TO_SOT_SMD:SOT-23-6 -> Package_DFN_QFN:VQFN-24-1EP_4x4mm_P0.5mm_EP2.5x2.5mm_ThermalVias
- moved R73 43.2 mm to (146.4, 98.8)
- moved R13 40.7 mm to (147.1, 96.4), turned to 180 degrees
- moved R26 37.7 mm to (148.1, 102.3)
- moved R19 36.9 mm to (149.7, 98.8), turned to -90 degrees
- moved JP13 36.7 mm to (149.0, 100.9), turned to -90 degrees
- moved R67 34.3 mm to (161.4, 94.1)
- moved C8 33.7 mm to (145.8, 90.5), turned to -90 degrees
- moved TP14 33.4 mm to (151.5, 101.5)
- moved R66 32.9 mm to (163.1, 94.2)
- moved U10 30.6 mm to (163.0, 90.8), turned to 0 degrees
- moved R25 30.1 mm to (182.3, 94.7)
- moved R21 29.8 mm to (178.8, 94.7)
- moved U4 28.8 mm to (153.3, 97.7), turned to 0 degrees
- moved C13 27.6 mm to (173.2, 94.7), turned to 180 degrees
- moved U11 27.5 mm to (206.3, 114.2), turned to 180 degrees
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Connections:
- net Net-(J12-Pin_3) renamed /3V3_unfused
- C8 pad 1: /12V_after_fuse -> /12V_input
- F9 pad 2: Net-(J12-Pin_2) -> /5V_unfused
- J12 pad 2: Net-(J12-Pin_2) -> /5V_unfused
- JP12 pad 2: Net-(D33-G) -> Net-(JP12-B)
- JP13 pad 1: /12V_after_fuse -> Net-(JP13-A)
- JP13 pad 2: Net-(JP13-B) -> GND
- Q1 pad 1: /12V_after_fuse -> Net-(Q1-G)
- Q1 pad 2: /12V_after_fuse -> Net-(Q1-D)
- Q1 pad 3: /12V_after_fuse -> +12VA
- R13 pad 1: /12V_after_fuse -> Net-(U4-SW)
- R13 pad 2: Net-(U4-INA+) -> SHUTOFF
- R14 pad 1: /12V_after_fuse -> Net-(Q3-D)
- R14 pad 2: Net-(Q1-G) -> Net-(Q1-D)
- R19 pad 1: Net-(U4-INA+) -> Net-(U4-SW)
- R19 pad 2: SHUTOFF -> Net-(U4-OV)
- R26 pad 1: SHUTOFF -> Net-(U4-OV)
- R26 pad 2: GND -> Net-(JP22-A)
- R65 pad 1: Net-(U4-OUTB) -> GND
- R65 pad 2: Net-(Q1-G) -> Net-(U4-TMR)
- R66 pad 1: Net-(U10-ADJ) -> Net-(U10-INBM)
- R66 pad 2: +5V -> Net-(U10-INAP)
- R67 pad 1: GND -> Net-(U10-INAP)
- R67 pad 2: Net-(U10-ADJ) -> GND
- R68 pad 1: +12VA -> /5V_unfused
- R68 pad 2: Net-(D33-G) -> Net-(U10-INBM)
- R73 pad 1: Net-(JP13-B) -> Net-(JP13-A)
- R73 pad 2: Net-(U4-INA+) -> GND
- TP10 pad 1: Net-(U4-OUTA) -> Net-(U4-INV_SLEEP)
- TP13 pad 1: Net-(U4-OUTB) -> Net-(U4-IMON)
- TP14 pad 1: SHUTOFF -> Net-(U4-EN)
- TP7 pad 1: /12V_after_fuse -> Net-(U4-INV_FLT)
- U10 pad 1: Net-(U10-ADJ) -> Net-(JP12-B)
- U10 pad 2: +5V -> GND
- U10 pad 3: +12VA -> Net-(U10-INAP)
- U11 pad 1: Net-(U11-REF) -> GND
- U11 pad 2: Net-(D33-G) -> +3V3
- U11 pad 3: GND -> +5V
- U4 pad 1: Net-(U4-OUTA) -> Net-(Q3-G)
- U4 pad 2: GND -> /12V_input
- U4 pad 3: Net-(U4-INA+) -> Net-(U4-SW)
- U4 pad 5: /12V_after_fuse -> Net-(U4-OV)
- U4 pad 6: Net-(U4-OUTB) -> Net-(U4-EN)
Routing:
- net /_8V: track 38.7 -> 82.4 mm, vias 1 -> 2
- net Net-(Q3-D): track 0.00 -> 32.8 mm, vias 0 -> 2
- net Net-(D26-K): track 0.00 -> 26.9 mm, vias 0 -> 2
- net Net-(J12-Pin_2): track 23.6 -> 0.00 mm, vias 1 -> 0
- net Net-(D33-G): track 21.9 -> 0.00 mm, vias 2 -> 0
- net /12V_after_fuse: track 19.1 -> 0.00 mm, vias 2 -> 0
- net Net-(JP12-B): track 0.00 -> 18.0 mm, vias 0 -> 2
- net Net-(Q3-G): track 0.00 -> 16.8 mm
- net Net-(Q1-D): track 0.00 -> 15.9 mm
- net Net-(Q1-G): track 3.94 -> 18.9 mm
- net /5V_unfused: track 0.00 -> 14.3 mm
- net SHUTOFF: track 9.51 -> 21.1 mm
- net /12V_input: track 0.00 -> 9.38 mm
- net Net-(JP22-A): track 0.00 -> 8.68 mm, vias 0 -> 1
- net Net-(U10-ADJ): track 8.49 -> 0.00 mm, vias 1 -> 0
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- removed copper zone on F.Cu, net /12V_after_fuse
Other:
- board text added: "RocciBoard V1.2"
- board text removed: "10A"
- board text removed: "Fuse"
- board text removed: "RocciBoard V1.1"
- board text removed: "TP10"
- board text removed: "TP13"
- board text removed: "TP14"
